File: motor-controller/motor-controller.sch (KiCad schematic (older format))
At the start: 36 parts, among them J1 Molex 172043-0201 R/A, J2 Molex 172043-0302 R/A, J3 MCU-IO, Q1 2N3904, U1 DRV10983PWP, U2 TLP291-4, U3 SI8600AC

Commit message: Added in isolator traces and placed resistors; need to add ground planes and tweak layout.
Parts:
- removed R12, R13: 4.7k, Resistor_SMD:R_0603_1608Metric, symbol Device:R_Small
- C7: value C -> 0.1u
- C8: value C -> 0.1u; footprint Capacitor_SMD:C_0201_0603Metric -> Capacitor_SMD:C_0603_1608Metric
- renumbered R14 to R12
Connections:
- net +3V3: now also U2.14, U2.5; no longer U2.12, U2.3
- net +5V: now also U2.12; no longer U2.14
- net DIR-MTR: now also U2.13; no longer U2.11
- net DIR-uC: now also U2.3; no longer U2.5
- net FG-MTR: now also U2.6; no longer U2.4
- net FG-uC: now also U2.11; no longer U2.13
- net at R4.1: now also U2.4; no longer U2.6
Other:
- moved on the sheet: R4, R5, R9, U2B
Changed lines of the file:
@@
 Text Label 10550 2700 0    50   ~ 0
 SPEED-MTR
-Text Label 9850 5650 0    50   ~ 0
+Text Label 9850 4350 0    50   ~ 0
 DIR-MTR
 Wire Wire Line
@@
 P 1200 6250
 F 0 "C7" H 1315 6296 50  0000 L CNN
-F 1 "C" H 1315 6205 50  0000 L CNN
+F 1 "0.1u" H 1315 6205 50  0000 L CNN
 F 2 "Capacitor_SMD:C_0603_1608Metric" H 1238 6100 50  0001 C CNN
 F 3 "~" H 1200 6250 50  0001 C CNN
@@
 	2400 5950 2100 5950
 $Comp
-L Device:R_Small R12
-U 1 1 6052FB90
-P 3850 6100
-F 0 "R12" H 3909 6146 50  0000 L CNN
-F 1 "4.7k" H 3909 6055 50  0000 L CNN
-F 2 "Resistor_SMD:R_0603_1608Metric" H 3850 6100 50  0001 C CNN
-F 3 "~" H 3850 6100 50  0001 C CNN
-	1    3850 6100
-	1    0    0    -1
-$EndComp
-$Comp
-L Device:R_Small R13
-U 1 1 6052FC18
-P 4150 6100
-F 0 "R13" H 4209 6146 50  0000 L CNN
-F 1 "4.7k" H 4209 6055 50  0000 L CNN
-F 2 "Resistor_SMD:R_0603_1608Metric" H 4150 6100 50  0001 C CNN
-F 3 "~" H 4150 6100 50  0001 C CNN
-	1    4150 6100
-	1    0    0    -1
-$EndComp
-Wire Wire Line
-	3700 5950 3850 5950
-Wire Wire Line
-	4150 5950 4150 6000
-Connection ~ 3700 5950
-Wire Wire Line
-	3850 6000 3850 5950
-Connection ~ 3850 5950
-Wire Wire Line
-	3850 5950 4150 5950
-Wire Wire Line
-	3600 6250 3850 6250
-Wire Wire Line
-	3850 6200 3850 6250
-Connection ~ 3850 6250
-Wire Wire Line
-	3600 6350 4150 6350
-Wire Wire Line
-	3850 6250 4450 6250
-Wire Wire Line
-	4150 6200 4150 6350
-Connection ~ 4150 6350
-Wire Wire Line
-	4150 6350 4450 6350
-$Comp
 L Isolator:TLP291-4 U2
 U 1 1 604C1323
@@
 L power:GNDD #PWR0120
 U 1 1 604C350F
-P 8950 6000
-F 0 "#PWR0120" H 8950 5750 50  0001 C CNN
-F 1 "GNDD" H 8954 5845 50  0000 C CNN
-F 2 "" H 8950 6000 50  0001 C CNN
-F 3 "" H 8950 6000 50  0001 C CNN
-	1    8950 6000
-	1    0    0    -1
-$EndComp
-Wire Wire Line
-	8950 5700 8950 5650
-Wire Wire Line
-	8950 5650 9050 5650
-Wire Wire Line
-	9050 5450 8900 5450
+P 8950 4700
+F 0 "#PWR0120" H 8950 4450 50  0001 C CNN
+F 1 "GNDD" H 8954 4545 50  0000 C CNN
+F 2 "" H 8950 4700 50  0001 C CNN
+F 3 "" H 8950 4700 50  0001 C CNN
+	1    8950 4700
+	1    0    0    -1
+$EndComp
+Wire Wire Line
+	8950 4400 8950 4350
+Wire Wire Line
+	8950 4350 9050 4350
+Wire Wire Line
+	9050 4150 8900 4150
 $Comp
 L power:+3V3 #PWR0121
 U 1 1 60551403
-P 9750 5350
-F 0 "#PWR0121" H 9750 5200 50  0001 C CNN
-F 1 "+3V3" H 9765 5523 50  0000 C CNN
-F 2 "" H 9750 5350 50  0001 C CNN
-F 3 "" H 9750 5350 50  0001 C CNN
-	1    9750 5350
-	1    0    0    -1
-$EndComp
-Wire Wire Line
-	9650 5650 9750 5650
-Wire Wire Line
-	9650 5450 9750 5450
-Wire Wire Line
-	9750 5450 9750 5350
+P 9750 4050
+F 0 "#PWR0121" H 9750 3900 50  0001 C CNN
+F 1 "+3V3" H 9765 4223 50  0000 C CNN
+F 2 "" H 9750 4050 50  0001 C CNN
+F 3 "" H 9750 4050 50  0001 C CNN
+	1    9750 4050
+	1    0    0    -1
+$EndComp
+Wire Wire Line
+	9650 4350 9750 4350
+Wire Wire Line
+	9650 4150 9750 4150
+Wire Wire Line
+	9750 4150 9750 4050
 $Comp
 L Device:R R5
 U 1 1 60559405
-P 9750 5850
-F 0 "R5" H 9820 5896 50  0000 L CNN
-F 1 "200" H 9820 5805 50  0000 L CNN
-F 2 "Resistor_SMD:R_0603_1608Metric" V 9680 5850 50  0001 C CNN
-F 3 "~" H 9750 5850 50  0001 C CNN
-	1    9750 5850
-	1    0    0    -1
-$EndComp
-Wire Wire Line
-	9750 6000 9750 6050
+P 9750 4550
+F 0 "R5" H 9820 4596 50  0000 L CNN
+F 1 "200" H 9820 4505 50  0000 L CNN
+F 2 "Resistor_SMD:R_0603_1608Metric" V 9680 4550 50  0001 C CNN
+F 3 "~" H 9750 4550 50  0001 C CNN
+	1    9750 4550
+	1    0    0    -1
+$EndComp
+Wire Wire Line
+	9750 4700 9750 4750
 $Comp
 L power:GND #PWR0122
 U 1 1 6055D350
-P 9750 6050
-F 0 "#PWR0122" H 9750 5800 50  0001 C CNN
-F 1 "GND" H 9755 5877 50  0000 C CNN
-F 2 "" H 9750 6050 50  0001 C CNN
-F 3 "" H 9750 6050 50  0001 C CNN
-	1    9750 6050
-	1    0    0    -1
-$EndComp
-Wire Wire Line
-	9750 5700 9750 5650
-Wire Wire Line
-	9750 5650 9850 5650
-Connection ~ 9750 5650
+P 9750 4750
+F 0 "#PWR0122" H 9750 4500 50  0001 C CNN
+F 1 "GND" H 9755 4577 50  0000 C CNN
+F 2 "" H 9750 4750 50  0001 C CNN
+F 3 "" H 9750 4750 50  0001 C CNN
+	1    9750 4750
+	1    0    0    -1
+$EndComp
+Wire Wire Line
+	9750 4400 9750 4350
+Wire Wire Line
+	9750 4350 9850 4350
+Connection ~ 9750 4350
 $Comp
 L power:GNDD #PWR0123
@@
 L power:GNDD #PWR0126
 U 1 1 6056E681
-P 9750 4800
-F 0 "#PWR0126" H 9750 4550 50  0001 C CNN
-F 1 "GNDD" H 9754 4645 50  0000 C CNN
-F 2 "" H 9750 4800 50  0001 C CNN
-F 3 "" H 9750 4800 50  0001 C CNN
-	1    9750 4800
-	1    0    0    -1
-$EndComp
-Wire Wire Line
-	8950 4400 9050 4400
-Wire Wire Line
-	9050 4200 8900 4200
+P 9750 6050
+F 0 "#PWR0126" H 9750 5800 50  0001 C CNN
+F 1 "GNDD" H 9754 5895 50  0000 C CNN
+F 2 "" H 9750 6050 50  0001 C CNN
+F 3 "" H 9750 6050 50  0001 C CNN
+	1    9750 6050
+	1    0    0    -1
+$EndComp
+Wire Wire Line
+	8950 5650 9050 5650
+Wire Wire Line
+	9050 5450 8900 5450
 $Comp
 L power:+3V3 #PWR0127
 U 1 1 6056E68A
-P 8900 4100
-F 0 "#PWR0127" H 8900 3950 50  0001 C CNN
-F 1 "+3V3" H 8915 4273 50  0000 C CNN
-F 2 "" H 8900 4100 50  0001 C CNN
-F 3 "" H 8900 4100 50  0001 C CNN
-	1    8900 4100
-	1    0    0    -1
-$EndComp
-Wire Wire Line
-	9650 4400 9750 4400
-Wire Wire Line
-	9650 4200 9750 4200
-Wire Wire Line
-	9750 4200 9750 4100
+P 8900 5350
+F 0 "#PWR0127" H 8900 5200 50  0001 C CNN
+F 1 "+3V3" H 8915 5523 50  0000 C CNN
+F 2 "" H 8900 5350 50  0001 C CNN
+F 3 "" H 8900 5350 50  0001 C CNN
+	1    8900 5350
+	1    0    0    -1
+$EndComp
+Wire Wire Line
+	9650 5650 9750 5650
+Wire Wire Line
+	9650 5450 9750 5450
+Wire Wire Line
+	9750 5450 9750 5350
 $Comp
 L Device:R R9
 U 1 1 6056E693
-P 9750 4600
-F 0 "R9" H 9820 4646 50  0000 L CNN
-F 1 "1k" H 9820 4555 50  0000 L CNN
-F 2 "Resistor_SMD:R_0603_1608Metric" V 9680 4600 50  0001 C CNN
-F 3 "~" H 9750 4600 50  0001 C CNN
-	1    9750 4600
-	1    0    0    -1
-$EndComp
-Wire Wire Line
-	9750 4750 9750 4800
-Wire Wire Line
-	9750 4450 9750 4400
-Wire Wire Line
-	9750 4400 9950 4400
-Connection ~ 9750 4400
+P 9750 5850
+F 0 "R9" H 9820 5896 50  0000 L CNN
+F 1 "1k" H 9820 5805 50  0000 L CNN
+F 2 "Resistor_SMD:R_0603_1608Metric" V 9680 5850 50  0001 C CNN
+F 3 "~" H 9750 5850 50  0001 C CNN
+	1    9750 5850
+	1    0    0    -1
+$EndComp
+Wire Wire Line
+	9750 6000 9750 6050
+Wire Wire Line
+	9750 5700 9750 5650
+Wire Wire Line
+	9750 5650 9950 5650
+Connection ~ 9750 5650
 $Comp
 L Device:R R8
@@
 L power:+5V #PWR0128
 U 1 1 605A5DFC
-P 9750 4100
-F 0 "#PWR0128" H 9750 3950 50  0001 C CNN
-F 1 "+5V" H 9765 4273 50  0000 C CNN
-F 2 "" H 9750 4100 50  0001 C CNN
-F 3 "" H 9750 4100 50  0001 C CNN
-	1    9750 4100
+P 9750 5350
+F 0 "#PWR0128" H 9750 5200 50  0001 C CNN
+F 1 "+5V" H 9765 5523 50  0000 C CNN
+F 2 "" H 9750 5350 50  0001 C CNN
+F 3 "" H 9750 5350 50  0001 C CNN
+	1    9750 5350
 	1    0    0    -1
 $EndComp
@@
 L Device:R R4
 U 1 1 60553263
-P 8950 5850
-F 0 "R4" H 9020 5896 50  0000 L CNN
-F 1 "75" H 9020 5805 50  0000 L CNN
-F 2 "Resistor_SMD:R_0603_1608Metric" V 8880 5850 50  0001 C CNN
-F 3 "~" H 8950 5850 50  0001 C CNN
-	1    8950 5850
+P 8950 4550
+F 0 "R4" H 9020 4596 50  0000 L CNN
+F 1 "75" H 9020 4505 50  0000 L CNN
+F 2 "Resistor_SMD:R_0603_1608Metric" V 8880 4550 50  0001 C CNN
+F 3 "~" H 8950 4550 50  0001 C CNN
+	1    8950 4550
 	1    0    0    -1
 $EndComp
@@
 L Isolator:TLP291-4 U2
 U 2 1 6057C93D
-P 9350 4300
-F 0 "U2" H 9350 4625 50  0000 C CNN
-F 1 "TLP291-4" H 9350 4534 50  0000 C CNN
-F 2 "Package_SO:SOIC-16_4.55x10.3mm_P1.27mm" H 9150 4100 50  0001 L CIN
-F 3 "https://toshiba.semicon-storage.com/info/docget.jsp?did=12858&prodName=TLP291-4" H 9350 4300 50  0001 L CNN
-	2    9350 4300
+P 9350 4250
+F 0 "U2" H 9350 4575 50  0000 C CNN
+F 1 "TLP291-4" H 9350 4484 50  0000 C CNN
+F 2 "Package_SO:SOIC-16_4.55x10.3mm_P1.27mm" H 9150 4050 50  0001 L CIN
+F 3 "https://toshiba.semicon-storage.com/info/docget.jsp?did=12858&prodName=TLP291-4" H 9350 4250 50  0001 L CNN
+	2    9350 4250
 	1    0    0    -1
 $EndComp
@@
 ======== Bidirectional I2C isolation ========
 Wire Wire Line
-	8900 4100 8900 4200
-Text Label 8950 4400 2    50   ~ 0
+	8900 5350 8900 5450
+Text Label 8950 5650 2    50   ~ 0
 FG-MTR
 Wire Wire Line
@@
 Wire Wire Line
 	2350 3450 2350 3500
-Text Label 9950 4400 1    50   ~ 0
+Text Label 9950 5650 1    50   ~ 0
 FG-uC
-Text Label 8900 5450 2    50   ~ 0
+Text Label 8900 4150 2    50   ~ 0
 DIR-uC
 Text Label 8900 2950 2    50   ~ 0
@@
 P 5250 6250
 F 0 "C8" H 5365 6296 50  0000 L CNN
-F 1 "C" H 5365 6205 50  0000 L CNN
-F 2 "Capacitor_SMD:C_0201_0603Metric" H 5288 6100 50  0001 C CNN
+F 1 "0.1u" H 5365 6205 50  0000 L CNN
+F 2 "Capacitor_SMD:C_0603_1608Metric" H 5288 6100 50  0001 C CNN
 F 3 "~" H 5250 6250 50  0001 C CNN
 	1    5250 6250
@@
 	6000 6300 6000 6400
 $Comp
-L Device:R R14
+L Device:R R12
 U 1 1 605F0B74
 P 6000 5750
-F 0 "R14" H 6070 5796 50  0000 L CNN
+F 0 "R12" H 6070 5796 50  0000 L CNN
 F 1 "220" H 6070 5705 50  0000 L CNN
 F 2 "Resistor_SMD:R_0603_1608Metric" V 5930 5750 50  0001 C CNN
@@
 Text Notes 6400 6300 0    50   ~ 0
 Motor controller power-indicator LED.\nIf illuminated, board is receiving \nhigh-voltage power.
+Wire Wire Line
+	3600 6350 4450 6350
+Wire Wire Line
+	3600 6250 4450 6250
 $EndSCHEMATC

Commit message: Preparation for fabrication.  Changed PCB silkscreen and added part numbers to schematic.
Added board description, version number, and date to PCB silkscreen.
Added Digi-Key part numbers and mating connectors as symbol attributes
for some connectors in schematic.
Parts:
- J1: Digi-Key part number (none) -> WM20737-ND
- J2: Connects to Molex no. 1726722003 --- https://www.digikey.com/en/product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 -> Molex no. 1726722003, 1726723003; Digi-Key part number (none) -> WM20740-ND
- J3: Connects to (none) -> JST XHP-7; Digi-Key part number (none) -> 455-2252-ND; Purchase link, Digi-Key https://www.digikey.com/en/products/detail/jst-sales-america-inc/B5B-XH-AM-LF-SN/1651037 -> https://www.digikey.com/en/products/detail/jst-sales-america-inc/B7B-XH-A-LF-SN/1651050
- L1: Digi-Key part number (none) -> 587-2956-6-ND
Changed lines of the file:
@@
 Sheet 1 1
 Title "Brushless DC Motor Controller"
-Date "2021-03-19"
-Rev "0.0.3"
+Date "2021-04-12"
+Rev "0.0.5"
 Comp "JHU Deliverbot Project"
 Comment1 "Drafted by @avnoks"
@@
 F 1 "47u" V 5313 1750 50  0000 C CNN
 F 2 "Inductor_SMD:L_Taiyo-Yuden_NR-60xx" H 5400 1750 50  0001 C CNN
-F 3 "~" H 5400 1750 50  0001 C CNN
+F 3 "https://ds.yuden.co.jp/TYCOMPAS/ut/detail?pn=NRS6045T470MMGK%20%20&u=M" H 5400 1750 50  0001 C CNN
 F 4 "https://www.digikey.com/en/products/detail/taiyo-yuden/NRS6045T470MMGK/2665994" V 5400 1750 50  0001 C CNN "Purchase link, Digi-Key"
+F 5 "587-2956-6-ND" V 5400 1750 50  0001 C CNN "Digi-Key part number"
 	1    5400 1750
 	0    1    1    0
@@
 F 2 "Connector_JST:JST_XH_B07B-XH-A_1x07_P2.50mm_Vertical" H 1100 5150 50  0001 C CNN
 F 3 "http://www.jst-mfg.com/product/pdf/eng/eXH.pdf" H 1100 5150 50  0001 C CNN
-F 4 "https://www.digikey.com/en/products/detail/jst-sales-america-inc/B5B-XH-AM-LF-SN/1651037" H 1100 5150 50  0001 C CNN "Purchase link, Digi-Key"
+F 4 "https://www.digikey.com/en/products/detail/jst-sales-america-inc/B7B-XH-A-LF-SN/1651050" H 1100 5150 50  0001 C CNN "Purchase link, Digi-Key"
+F 5 "455-2252-ND" H 1100 5150 50  0001 C CNN "Digi-Key part number"
+F 6 "JST XHP-7" H 1100 5150 50  0001 C CNN "Connects to"
 	1    1100 5150
 	1    0    0    -1
@@
 F 2 "custom:172043-0302_MOL" H 5850 2500 50  0001 C CNN
 F 3 "https://www.molex.com/pdm_docs/sd/1720430302_sd.pdf" H 5850 2500 50  0001 C CNN
-F 4 "Molex no. 1726722003 --- https://www.digikey.com/en/products/detail/molex/1726722003/5154604" H 5850 2500 50  0001 C CNN "Connects to"
+F 4 "Molex no. 1726722003, 1726723003" H 5850 2500 50  0001 C CNN "Connects to"
 F 5 "https://www.digikey.com/en/products/detail/molex/1720430302/4839872" H 5850 2500 50  0001 C CNN "Purchase link, Digi-Key"
+F 6 "WM20740-ND" H 5850 2500 50  0001 C CNN "Digi-Key part number"
 	1    5850 2500
 	1    0    0    1
@@
 F 4 "Molex 1726722002 --- https://www.digikey.com/en/products/detail/molex/1726722002/5154603" H 1900 1700 50  0001 C CNN "Connects with"
 F 5 "https://www.digikey.com/en/products/detail/molex/1720430201/4839863" H 1900 1700 50  0001 C CNN "Purchase link, Digi-Key"
+F 6 "WM20737-ND" H 1900 1700 50  0001 C CNN "Digi-Key part number"
 	1    1900 1700
 	1    0    0    1
