File: PMS/PMS/PMS.kicad_sch (KiCad schematic)
At the start: 36 parts, among them IC1 TMCS1107A1BQDRQ1, IC2 ADR3450ARJZ-R7, IC3 TL2575-12IKTTR, J1 XT60PW-M, J2 XT60PW-F, J3 XT60PW-M, J4 XT60PW-F, J5 XT60PW-F, J6 Conn_01x03_Male, J7 Conn_01x02_Male, J8 Conn_01x02_Male, U1 ADC101C027CIMK, U2 ADC101C027CIMK, U3 LA12-48V21

Commit message: Layout complete.
Parts:
- added H1, H2, H3, H4: MountingHole, MountingHole:MountingHole_3.2mm_M3_ISO14580, symbol Mechanical:MountingHole
- added JP1: Jumper_2_Bridged, Jumper:SolderJumper-2_P1.3mm_Bridged2Bar_Pad1.0x1.5mm, symbol Jumper:Jumper_2_Bridged
Connections:
- net +24V: no longer J2.2 (+), R1.1
- net +5V: now also C7.1, C8.1, IC2.3 (EN), IC2.4 (VIN)
- net +5VP: no longer C7.1, C8.1, IC2.3 (EN), IC2.4 (VIN)
- net 24V_OUT: now also J2.2 (+), R1.1
- net GND: now also JP1.1 (A); no longer C1.2, C2.2, C3.2, C4.2, C5.2, C6.1, IC1.5 (GND), IC2.1 (GND_FORCE), IC2.2 (GND_SEN), R3.2, U1.2 (GND), U1.4 (ADDR), U2.2 (GND)
- new net GNDA: C1.2, C2.2, C3.2, C4.2, C5.2, C6.1, IC1.5 (GND), IC2.1 (GND_FORCE), IC2.2 (GND_SEN), JP1.2 (B), R3.2, U1.2 (GND), U1.4 (ADDR), U2.2 (GND)
