File: PMS/PMS/PMS.kicad_pcb (KiCad board)
At the start: 2 copper layers, 27 parts, among them IC1 TMCS1107A1BQDRQ1, IC2 ADR3450ARJZ-R7, J1 XT60PW-M, J2 XT60PW-F, J3 XT60PW-M, J4 XT60PW-F, J5 XT60PW-F, J6 Conn_01x03_Male, J7 Conn_01x02_Male, U1 ADC101C027CIMK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

Commit message: Layout complete.
Parts:
- added H1: MountingHole, MountingHole:MountingHole_3.2mm_M3_ISO14580, F.Cu at (60.0, 52.0)
- added H2: MountingHole, MountingHole:MountingHole_3.2mm_M3_ISO14580, F.Cu at (135.0, 52.0)
- added H3: MountingHole, MountingHole:MountingHole_3.2mm_M3_ISO14580, F.Cu at (60.0, 102.0)
- added H4: MountingHole, MountingHole:MountingHole_3.2mm_M3_ISO14580, F.Cu at (135.0, 102.0)
- added JP1: Jumper_2_Bridged, Jumper:SolderJumper-2_P1.3mm_Bridged2Bar_Pad1.0x1.5mm, F.Cu at (101.8, 74.2)
- moved J7 116.5 mm to (66.5, 54.8), turned to 90 degrees
- moved R4 115.0 mm to (102.5, 92.5), turned to 90 degrees
- moved R2 102.1 mm to (98.5, 74.2)
- moved C6 98.5 mm to (93.0, 79.4), turned to 180 degrees
- moved R1 97.8 mm to (97.8, 71.2), turned to -90 degrees
- moved C8 97.3 mm to (93.4, 71.4), turned to 180 degrees
- moved C7 96.4 mm to (93.4, 73.7), turned to 180 degrees
- moved R3 76.2 mm to (100.2, 92.5), turned to 90 degrees
- moved C5 74.6 mm to (107.2, 88.8)
- moved J1 74.5 mm to (122.0, 97.2), turned to 180 degrees
- moved IC2 69.6 mm to (93.3, 76.3), turned to 180 degrees
- moved F1 65.6 mm to (121.0, 90.1), turned to 90 degrees
- moved C1 55.7 mm to (107.9, 79.6), turned to -90 degrees
- moved C4 54.2 mm to (99.8, 88.8)
- moved R6 51.5 mm to (105.2, 96.8)
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Connections:
- C1 pad 2: GND -> GNDA
- C2 pad 2: GND -> GNDA
- C3 pad 2: GND -> GNDA
- C4 pad 2: GND -> GNDA
- C5 pad 2: GND -> GNDA
- C6 pad 1: GND -> GNDA
- C7 pad 1: +5VP -> +5V
- C8 pad 1: +5VP -> +5V
- IC1 pad 5: GND -> GNDA
- IC2 pad 1: GND -> GNDA
- IC2 pad 2: GND -> GNDA
- IC2 pad 3: +5VP -> +5V
- IC2 pad 4: +5VP -> +5V
- J2 pad 2: +24V -> 24V_OUT
- R1 pad 1: +24V -> 24V_OUT
- R3 pad 2: GND -> GNDA
- U1 pad 2: GND -> GNDA
- U1 pad 4: GND -> GNDA
- U2 pad 2: GND -> GNDA
Routing:
- net +5VP: track 0.00 -> 27.4 mm
- net +5VA: track 0.00 -> 25.5 mm, vias 0 -> 7
- net Net-(R1-Pad2): track 0.00 -> 19.7 mm
- net GNDA: track 0.00 -> 19.5 mm, vias 0 -> 13
- net SDA: track 0.00 -> 16.3 mm, vias 0 -> 2
- net Net-(IC1-Pad7): track 0.00 -> 16.1 mm
- net SCL: track 0.00 -> 16.1 mm
- net +BATT: track 0.00 -> 8.23 mm
- net +5V: track 0.00 -> 7.67 mm, vias 0 -> 1
- net GND: track 0.00 -> 5.06 mm, vias 0 -> 4
- net Net-(R3-Pad1): track 0.00 -> 4.11 mm
- net 24V_OUT: vias 0 -> 13
- net +24V: vias 0 -> 13
- added copper zone on B.Cu, net +24V
- added copper zone on F.Cu, net +24V
- added copper zone on In2.Cu, net +5V
- added copper zone on In2.Cu, net +5VA
- added copper zone on B.Cu, net 24V_OUT
- added copper zone on F.Cu, net 24V_OUT
- added copper zone on In1.Cu, net GND
- added copper zone on In1.Cu, net GNDA
Other:
- board outline added: 82.5 x 57.5 mm
- copper layers 2 -> 4

Commit message: cleanup
Routing:
- net +5VA: track 25.5 -> 24.3 mm
- net SCL: track 16.1 -> 15.3 mm
Changed lines of the file:
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@@
   )
   (segment (start 106.25 86.375) (end 106.25 88.675) (width 1) (layer "F.Cu") (net 1))
-  (segment (start 98.45 89.0125) (end 98.7125 88.75) (width 0.5) (layer "F.Cu") (net 1))
-  (segment (start 107.905 78.5575) (end 107.9 78.5625) (width 0.5) (layer "F.Cu") (net 1))
   (segment (start 98.7125 88.75) (end 98.7125 86.475) (width 1) (layer "F.Cu") (net 1))
-  (segment (start 98.7125 86.475) (end 98.75 86.4375) (width 1) (layer "F.Cu") (net 1))
   (segment (start 106.2 91.3625) (end 106.2 88.775) (width 0.5) (layer "F.Cu") (net 1))
-  (segment (start 106.3 96.8) (end 106.25 96.75) (width 1) (layer "F.Cu") (net 1))
-  (segment (start 106.325 86.3) (end 106.25 86.375) (width 1) (layer "F.Cu") (net 1))
-  (segment (start 107.9625 78.5) (end 107.9 78.5625) (width 1) (layer "F.Cu") (net 1))
-  (segment (start 106.25 88.675) (end 106.175 88.75) (width 1) (layer "F.Cu") (net 1))
   (segment (start 107.905 76.211) (end 107.905 78.5575) (width 0.5) (layer "F.Cu") (net 1))
   (segment (start 98.4 96.7) (end 99.7 96.7) (width 1) (layer "F.Cu") (net 1))
   (segment (start 102.5 90.2) (end 102.5 91.5) (width 1) (layer "F.Cu") (net 1))
-  (segment (start 106.2 88.775) (end 106.175 88.75) (width 0.5) (layer "F.Cu") (net 1))
   (segment (start 92.0408 76.28195) (end 92.0408 77.22175) (width 0.5) (layer "F.Cu") (net 1))
   (segment (start 107.5 96.8) (end 106.3 96.8) (width 1) (layer "F.Cu") (net 1))
-  (segment (start 99.7 96.7) (end 99.75 96.75) (width 1) (layer "F.Cu") (net 1))
   (segment (start 100.2 86.3) (end 98.8875 86.3) (width 1) (layer "F.Cu") (net 1))
   (segment (start 98.45 91.3625) (end 98.45 89.0125) (width 0.5) (layer "F.Cu") (net 1))
   (segment (start 92.0408 77.22175) (end 92.0408 79.3592) (width 0.5) (layer "F.Cu") (net 1))
-  (segment (start 92.0408 79.44705) (end 92.0125 79.41875) (width 1) (layer "F.Cu") (net 1))
   (segment (start 107.8 86.3) (end 106.325 86.3) (width 1) (layer "F.Cu") (net 1))
   (segment (start 92.0408 80.9) (end 92.0408 79.44705) (width 1) (layer "F.Cu") (net 1))
-  (segment (start 92.0408 79.3592) (end 92.0408 79.39045) (width 0.5) (layer "F.Cu") (net 1))
   (segment (start 109.3 78.5) (end 107.9625 78.5) (width 1) (layer "F.Cu") (net 1))
-  (segment (start 98.8875 86.3) (end 98.75 86.4375) (width 1) (layer "F.Cu") (net 1))
   (via (at 107.8 86.3) (size 0.8) (drill 0.4) (layers "F.Cu" "B.Cu") (free) (net 1))
   (via (at 100.2 86.3) (size 0.8) (drill 0.4) (layers "F.Cu" "B.Cu") (free) (net 1))
@@
   (segment (start 94.4792 75.34215) (end 94.4792 73.71045) (width 0.5) (layer "F.Cu") (net 6))
   (segment (start 95.75 71.5) (end 94.51875 71.5) (width 1) (layer "F.Cu") (net 6))
-  (segment (start 94.51875 71.5) (end 94.4375 71.41875) (width 1) (layer "F.Cu") (net 6))
   (segment (start 92.0408 75.34215) (end 94.4792 75.34215) (width 0.5) (layer "F.Cu") (net 6))
   (via (at 95.75 71.5) (size 0.8) (drill 0.4) (layers "F.Cu" "B.Cu") (free) (net 6))
@@
   (segment (start 106.2 93.6375) (end 106.2 94.8) (width 0.25) (layer "F.Cu") (net 10))
   (segment (start 99.23702 94.42452) (end 98.45 93.6375) (width 0.25) (layer "F.Cu") (net 10))
-  (segment (start 104.1 96.6) (end 104.25 96.75) (width 0.25) (layer "F.Cu") (net 10))
   (segment (start 103 96.6) (end 104.1 96.6) (width 0.25) (layer "F.Cu") (net 10))
   (via (at 101.65 95.25) (size 0.8) (drill 0.4) (layers "F.Cu" "B.Cu") (net 10))
@@
   (segment (start 100.3 95.3) (end 98.778928 95.3) (width 0.25) (layer "F.Cu") (net 11))
   (segment (start 101.75 96.75) (end 100.3 95.3) (width 0.25) (layer "F.Cu") (net 11))
-  (segment (start 105.25 93.6375) (end 105.25 94.021072) (width 0.25) (layer "F.Cu") (net 11))
   (segment (start 105.25 94.021072) (end 104.646552 94.62452) (width 0.25) (layer "F.Cu") (net 11))
   (segment (start 101.75 102.025) (end 101.75 96.75) (width 1) (layer "F.Cu") (net 11))
   (segment (start 98.778928 95.3) (end 97.5 94.021072) (width 0.25) (layer "F.Cu") (net 11))
   (segment (start 103.82548 94.62452) (end 101.75 96.7) (width 0.25) (layer "F.Cu") (net 11))
-  (segment (start 97.5 94.021072) (end 97.5 93.6375) (width 0.25) (layer "F.Cu") (net 11))
-  (segment (start 101.75 96.7) (end 101.75 96.75) (width 0.25) (layer "F.Cu") (net 11))
   (segment (start 104.646552 94.62452) (end 103.82548 94.62452) (width 0.25) (layer "F.Cu") (net 11))
   (segment (start 97.12548 88.62452) (end 97.12548 74.71202) (width 1) (layer "F.Cu") (net 13))
@@
   (segment (start 97.75 74.0875) (end 97.75 72.25) (width 1) (layer "F.Cu") (net 13))
   (segment (start 104.3 93.6375) (end 102.6375 93.6375) (width 0.5) (layer "F.Cu") (net 14))
-  (segment (start 102.6375 93.6375) (end 102.5 93.5) (width 0.5) (layer "F.Cu") (net 14))
   (segment (start 100.25 93.5) (end 102.5 93.5) (width 1) (layer "F.Cu") (net 14))
   (segment (start 100.25 90.5) (end 100.5 90.25) (width 1) (layer "F.Cu") (net 15))
@@
   (segment (start 101.75 74.9) (end 101.75 76.25) (width 1) (layer "F.Cu") (net 15))
   (segment (start 94.4792 77.22175) (end 95.853 77.22175) (width 0.5) (layer "F.Cu") (net 15))
-  (segment (start 107.9625 80.7) (end 107.9 80.6375) (width 1) (layer "F.Cu") (net 15))
   (segment (start 108.25 88.75) (end 108.25 87.5) (width 1) (layer "F.Cu") (net 15))
   (segment (start 100.7875 88.75) (end 100.7875 89.9625) (width 1) (layer "F.Cu") (net 15))
@@
   (segment (start 104.095 77.695) (end 104.1 77.7) (width 0.5) (layer "F.Cu") (net 15))
   (segment (start 97.5 91.3625) (end 97.5 90) (width 0.5) (layer "F.Cu") (net 15))
-  (segment (start 98.8125 83.5) (end 98.75 83.5625) (width 1) (layer "F.Cu") (net 15))
   (segment (start 107.75 83.5) (end 106.25 83.5) (width 1) (layer "F.Cu") (net 15))
   (segment (start 104.095 76.211) (end 104.095 77.695) (width 0.5) (layer "F.Cu") (net 15))

Commit message: all traces now routed on the topmost layer
Routing:
- net SDA: track 16.1 -> 19.0 mm, vias 2 -> 0
Changed lines of the file:
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@@
   (via (at 92.0408 80.9) (size 0.8) (drill 0.4) (layers "F.Cu" "B.Cu") (net 1))
   (via (at 102.5 90.2) (size 0.8) (drill 0.4) (layers "F.Cu" "B.Cu") (free) (net 1))
+  (segment (start 99.4125 72.8625) (end 99.4125 74.25) (width 1) (layer "F.Cu") (net 2))
   (segment (start 101.75 73.6) (end 101.75 72.25) (width 1) (layer "F.Cu") (net 2))
-  (segment (start 99.5 73) (end 99.5 74.1625) (width 1) (layer "F.Cu") (net 2))
+  (segment (start 99.4 72.85) (end 99.4125 72.8625) (width 1) (layer "F.Cu") (net 2))
   (segment (start 92.3625 73.66875) (end 91.15 73.66875) (width 1) (layer "F.Cu") (net 2))
-  (segment (start 99.5 74.1625) (end 99.4125 74.25) (width 1) (layer "F.Cu") (net 2))
   (segment (start 91.15 71.41875) (end 92.3625 71.41875) (width 1) (layer "F.Cu") (net 2))
   (via (at 91.15 71.41875) (size 0.8) (drill 0.4) (layers "F.Cu" "B.Cu") (free) (net 2))
   (via (at 101.75 72.25) (size 0.8) (drill 0.4) (layers "F.Cu" "B.Cu") (free) (net 2))
-  (via (at 99.5 73) (size 0.8) (drill 0.4) (layers "F.Cu" "B.Cu") (free) (net 2))
+  (via (at 99.4 72.85) (size 0.8) (drill 0.4) (layers "F.Cu" "B.Cu") (free) (net 2))
   (via (at 91.15 73.66875) (size 0.8) (drill 0.4) (layers "F.Cu" "B.Cu") (free) (net 2))
   (segment (start 65 82.9) (end 67.776282 82.9) (width 5) (layer "F.Cu") (net 3))
@@
   (segment (start 106.635 80.865) (end 104.3 83.2) (width 0.5) (layer "F.Cu") (net 9))
   (segment (start 106.635 76.211) (end 106.635 80.865) (width 0.5) (layer "F.Cu") (net 9))
-  (segment (start 100.82452 94.42452) (end 99.23702 94.42452) (width 0.25) (layer "F.Cu") (net 10))
+  (segment (start 106.2 92.7) (end 106 92.5) (width 0.25) (layer "F.Cu") (net 10))
   (segment (start 104.25 102.025) (end 104.25 96.75) (width 1) (layer "F.Cu") (net 10))
-  (segment (start 101.65 95.25) (end 100.82452 94.42452) (width 0.25) (layer "F.Cu") (net 10))
+  (segment (start 106.2 93.6375) (end 106.2 92.7) (width 0.25) (layer "F.Cu") (net 10))
+  (segment (start 98.45 92.75) (end 98.45 93.6375) (width 0.25) (layer "F.Cu") (net 10))
+  (segment (start 106 92.5) (end 98.7 92.5) (width 0.25) (layer "F.Cu") (net 10))
   (segment (start 106.2 94.8) (end 104.25 96.75) (width 0.25) (layer "F.Cu") (net 10))
   (segment (start 106.2 93.6375) (end 106.2 94.8) (width 0.25) (layer "F.Cu") (net 10))
-  (segment (start 99.23702 94.42452) (end 98.45 93.6375) (width 0.25) (layer "F.Cu") (net 10))
-  (segment (start 103 96.6) (end 104.1 96.6) (width 0.25) (layer "F.Cu") (net 10))
-  (via (at 101.65 95.25) (size 0.8) (drill 0.4) (layers "F.Cu" "B.Cu") (net 10))
-  (via (at 103 96.6) (size 0.8) (drill 0.4) (layers "F.Cu" "B.Cu") (net 10))
-  (segment (start 101.65 95.25) (end 103 96.6) (width 0.25) (layer "B.Cu") (net 10))
+  (segment (start 98.7 92.5) (end 98.45 92.75) (width 0.25) (layer "F.Cu") (net 10))
+  (segment (start 104.021072 95.25) (end 103.2 95.25) (width 0.25) (layer "F.Cu") (net 11))
   (segment (start 100.3 95.3) (end 98.778928 95.3) (width 0.25) (layer "F.Cu") (net 11))
   (segment (start 101.75 96.75) (end 100.3 95.3) (width 0.25) (layer "F.Cu") (net 11))
-  (segment (start 105.25 94.021072) (end 104.646552 94.62452) (width 0.25) (layer "F.Cu") (net 11))
+  (segment (start 103.2 95.25) (end 101.75 96.7) (width 0.25) (layer "F.Cu") (net 11))
   (segment (start 101.75 102.025) (end 101.75 96.75) (width 1) (layer "F.Cu") (net 11))
   (segment (start 98.778928 95.3) (end 97.5 94.021072) (width 0.25) (layer "F.Cu") (net 11))
-  (segment (start 103.82548 94.62452) (end 101.75 96.7) (width 0.25) (layer "F.Cu") (net 11))
-  (segment (start 104.646552 94.62452) (end 103.82548 94.62452) (width 0.25) (layer "F.Cu") (net 11))
+  (segment (start 105.25 94.021072) (end 104.021072 95.25) (width 0.25) (layer "F.Cu") (net 11))
   (segment (start 97.12548 88.62452) (end 97.12548 74.71202) (width 1) (layer "F.Cu") (net 13))
   (segment (start 96.55 89.3) (end 96.55 91.3625) (width 0.5) (layer "F.Cu") (net 13))
@@
   (segment (start 101.75 74.9) (end 101.75 76.25) (width 1) (layer "F.Cu") (net 15))
   (segment (start 94.4792 77.22175) (end 95.853 77.22175) (width 0.5) (layer "F.Cu") (net 15))
-  (segment (start 108.25 88.75) (end 108.25 87.5) (width 1) (layer "F.Cu") (net 15))
   (segment (start 100.7875 88.75) (end 100.7875 89.9625) (width 1) (layer "F.Cu") (net 15))
   (segment (start 94.4792 76.28195) (end 95.8868 76.28195) (width 0.5) (layer "F.Cu") (net 15))
   (segment (start 99.9 83.5) (end 98.8125 83.5) (width 1) (layer "F.Cu") (net 15))
+  (segment (start 108.25 88.75) (end 108.25 90.25) (width 1) (layer "F.Cu") (net 15))
   (segment (start 104.095 77.695) (end 104.1 77.7) (width 0.5) (layer "F.Cu") (net 15))
   (segment (start 97.5 91.3625) (end 97.5 90) (width 0.5) (layer "F.Cu") (net 15))
@@
   (segment (start 100.7875 89.9625) (end 100.5 90.25) (width 1) (layer "F.Cu") (net 15))
   (via (at 97.5 90) (size 0.8) (drill 0.4) (layers "F.Cu" "B.Cu") (free) (net 15))
-  (via (at 108.25 87.5) (size 0.8) (drill 0.4) (layers "F.Cu" "B.Cu") (free) (net 15))
+  (via (at 108.25 90.25) (size 0.8) (drill 0.4) (layers "F.Cu" "B.Cu") (free) (net 15))
   (via (at 100.5 90.25) (size 0.8) (drill 0.4) (layers "F.Cu" "B.Cu") (free) (net 15))
   (via (at 101.75 76.25) (size 0.8) (drill 0.4) (layers "F.Cu" "B.Cu") (free) (net 15))
