File: IR-Breakout/IR-Breakout.kicad_pcb (KiCad board)
At the start: 2 copper layers, 18 x 18 mm, 13 parts, among them J1 PWR, J2 I2C, U1 LDK120M18R, U2 TMD37253M

Commit message: corrected values for pullups on SDA, SCL, and INT
Parts:
- R1: value 4.7u -> 22
- R2, R3, R4: value 4.7u -> 10K
Connections:
- net Net-(J2-Pad1) renamed /SDA
- net Net-(J2-Pad2) renamed /SCL
- net Net-(J2-Pad3) renamed /INT
- U2 pad 5: Net-(U2-Pad5) -> unconnected-(U2-Pad5)
Other:
- net class Default removed
- net class Power removed
